Commit message: fixed line following to be more stable, created state machine, installed lidar

File: src/2025_competition/robbie/urdf/robbie.xacro (robot description, xacro)
@@ -12,4 +12,7 @@
   <xacro:property name="wheel_width" value="0.03"/>
   <xacro:property name="wheel_mass" value="0.025"/>
+  <xacro:property name="lidar_radius" value="0.02"/>
+  <xacro:property name="lidar_height" value="0.01"/>
+  <xacro:property name="lidar_mass" value="0.01"/>
   <xacro:include filename="$(find robbie)/urdf/macros.xacro"/>
   <xacro:include filename="$(find robbie)/urdf/materials.xacro"/>
@@ -105,4 +108,18 @@
     </visual>
   </link>
+  <link name='lidar_link'>
+    <xacro:cylinder_inertial name="lidar_link" m="${lidar_mass}" r="${lidar_radius}" h="${lidar_height}"/>
+    <collision name='lidar_link_collision'>
+      <geometry>
+        <cylinder radius="${lidar_radius}" length="${lidar_height}"/>
+      </geometry>
+    </collision>
+    <visual name='lidar_link_visual'>
+      <origin xyz="0 0 0" rpy="0 0 0"/>
+      <geometry>
+        <cylinder radius="${lidar_radius}" length="${lidar_height}"/>
+      </geometry>
+    </visual>
+  </link>
   <joint name="wheel_FR_joint" type="continuous">
     <parent link="chassis"/>
@@ -138,4 +155,9 @@
     <origin xyz="${chassis_length/2} 0 ${chassis_height/2+camera_height/2}"/>
   </joint>
+  <joint name="lidar_joint" type="fixed">
+    <parent link="chassis"/>
+    <child link="lidar_link"/>
+    <origin xyz="${chassis_length/2} 0 ${chassis_height/2 - camera_height/2 - lidar_height/2}" rpy="0 0 0"/>
+  </joint>
   <gazebo reference="chassis">
     <material>Gazebo/Orange</material>
@@ -143,4 +165,7 @@
   <gazebo reference="camera_link">
     <material>Gazebo/Blue</material>
+  </gazebo>
+   <gazebo reference="camera_link">
+    <material>Gazebo/Black</material>
   </gazebo>
   <gazebo reference="wheel_FL">
@@ -175,5 +200,5 @@
       <update_rate>30.0</update_rate>
       <camera name="head">
-        <horizontal_fov>1.3962634</horizontal_fov>
+        <horizontal_fov>1.57</horizontal_fov>
         <image>
           <width>800</width>
@@ -210,3 +235,34 @@
     </sensor>
   </gazebo>
+   <gazebo reference="lidar_link">
+    <sensor type="ray" name="head_hokuyo_sensor">
+      <pose>0 0 0 0 0 0</pose>
+      <visualize>true</visualize>
+      <update_rate>30</update_rate>
+      <ray>
+        <scan>
+          <horizontal>
+            <samples>720</samples>
+            <resolution>1</resolution>
+            <min_angle>-1.57</min_angle>
+            <max_angle>1.57</max_angle>
+          </horizontal>
+        </scan>
+        <range>
+          <min>0.035</min>
+          <max>.5</max>
+          <resolution>0.01</resolution>
+        </range>
+        <noise>
+          <type>gaussian</type>
+          <mean>0.0</mean>
+          <stddev>0.01</stddev>
+        </noise>
+      </ray>
+      <plugin name="gazebo_ros_head_hokuyo_controller" filename="libgazebo_ros_laser.so">
+        <topicName>/scan</topicName>
+        <frameName>lidar_link</frameName>
+      </plugin>
+    </sensor>
+  </gazebo>
 </robot>
